Commit message: 机械臂

File: model/myrobotv52.urdf (robot description, URDF)
Before this commit: robot vehicle_blue, 7 links, 6 joints
Links:
- added link arm_yaw_link, mass 0.6; collision cylinder length=0.10 radius=0.04; visual cylinder length=0.10 radius=0.04
- added link forearm_link, mass 0.6; collision cylinder length=0.60 radius=0.03; visual cylinder length=0.60 radius=0.03
- added link suction_cup_link, mass 0.1; collision cylinder length=0.05 radius=0.06; visual cylinder length=0.05 radius=0.06
- added link upper_arm_link, mass 0.8; collision cylinder length=0.60 radius=0.035; visual cylinder length=0.60 radius=0.035
- added link wrist_link, mass 0.25; collision cylinder length=0.20 radius=0.025; visual cylinder length=0.20 radius=0.025
Joints:
- added joint joint1_base_yaw: type revolute, parent base_link, child arm_yaw_link, origin xyz=-0.15 0 0.0835 rpy=0 0 0, axis 0 0 1, limit lower=-3.1415926 upper=3.1415926 effort=50 velocity=5
- added joint joint2_shoulder_pitch: type revolute, parent arm_yaw_link, child upper_arm_link, origin xyz=0 0 0.10 rpy=0 0 0, axis 0 1 0, limit lower=-2.0 upper=2.0 effort=50 velocity=5
- added joint joint3_elbow_pitch: type revolute, parent upper_arm_link, child forearm_link, origin xyz=0 0 0.60 rpy=0 0 0, axis 0 1 0, limit lower=-2.0 upper=2.0 effort=50 velocity=5
- added joint joint4_wrist_pitch: type revolute, parent forearm_link, child wrist_link, origin xyz=0 0 0.60 rpy=0 0 0, axis 0 1 0, limit lower=-2.0 upper=2.0 effort=50 velocity=5
- added joint suction_fixed_joint: type fixed, parent wrist_link, child suction_cup_link, origin xyz=0 0 0.20 rpy=0 0 0

Commit message: 重新设计机械臂

File: model/myrobotv52.urdf (robot description, URDF)
Before this commit: robot vehicle_blue, 12 links, 11 joints
Links:
- removed link arm_yaw_link
- removed link forearm_link
- removed link suction_cup_link
- removed link upper_arm_link
- removed link wrist_link
- added link arm_extend_forearm, mass 0.5; collision box size=0.3 0.05 0.05; visual box size=0.3 0.05 0.05
- added link arm_rot_base, mass 0.8; collision cylinder length=0.09 radius=0.07; visual cylinder length=0.09 radius=0.07
- added link arm_upper_link, mass 0.7; collision box size=0.4 0.06 0.06; visual box size=0.4 0.06 0.06
- added link arm_wrist_rot, mass 0.3; collision box size=0.08 0.08 0.08; visual box size=0.08 0.08 0.08
- added link finger_1, mass 0.05; collision box size=0.1 0.02 0.02; visual box size=0.1 0.02 0.02
- added link finger_2, mass 0.05; collision box size=0.1 0.02 0.02; visual box size=0.1 0.02 0.02
- added link finger_3, mass 0.05; collision box size=0.1 0.02 0.02; visual box size=0.1 0.02 0.02
- added link gripper_base, mass 0.2; collision box size=0.05 0.15 0.15; visual box size=0.05 0.15 0.15
- added link lift_base, mass 1.2; collision box size=0.12 0.12 0.2; visual box size=0.12 0.12 0.2
- added link lift_platform, mass 1; collision box size=0.3 0.25 0.08; visual box size=0.3 0.25 0.08
- added link lift_slide, mass 2; collision box size=0.08 0.08 1.2; visual box size=0.08 0.08 1
Joints:
- removed joint joint1_base_yaw
- removed joint joint2_shoulder_pitch
- removed joint joint3_elbow_pitch
- removed joint joint4_wrist_pitch
- removed joint suction_fixed_joint
- added joint arm_forearm_extend_joint: type prismatic, parent arm_upper_link, child arm_extend_forearm, origin xyz=0 0 0.363 rpy=0 0 0, axis 1 0 0, limit lower=0 upper=0.3 effort=80 velocity=0.25
- added joint arm_rot_joint: type revolute, parent lift_platform, child arm_rot_base, origin xyz=0 0 0.115 rpy=0 0 0, axis 0 0 1, limit lower=-3.14 upper=3.14 effort=150 velocity=1.2
- added joint arm_upper_pitch_joint: type revolute, parent arm_rot_base, child arm_upper_link, origin xyz=0 0 0.09 rpy=0 0 0, axis 0 1 0, limit lower=-0.785 upper=1.57 effort=120 velocity=1
- added joint finger1_joint: type revolute, parent gripper_base, child finger_1, origin xyz=0 0.04 -0.07 rpy=0 0 0, axis 0 1 0, limit lower=-0.6 upper=0.6 effort=15 velocity=2
- added joint finger2_joint: type revolute, parent gripper_base, child finger_2, origin xyz=0 -0.04 -0.07 rpy=0 0 0, axis 0 1 0, limit lower=-0.6 upper=0.6 effort=15 velocity=2
- added joint finger3_joint: type revolute, parent gripper_base, child finger_3, origin xyz=0 0 0.05 rpy=0 0 0, axis 0 1 0, limit lower=-0.6 upper=0.6 effort=15 velocity=2
- added joint gripper_fixed_joint: type fixed, parent arm_wrist_rot, child gripper_base, origin xyz=0.06 0 0 rpy=-3.1415926 0 -3.1415926
- added joint lift_base_joint: type fixed, parent base_link, child lift_base, origin xyz=-0.25 0 0.167 rpy=0 0 0
- added joint lift_slide_joint: type fixed, parent base_link, child lift_slide, origin xyz=-0.25 0 0.167 rpy=0 0 0
- added joint platform_joint: type prismatic, parent lift_slide, child lift_platform, origin xyz=0 0 0.333 rpy=0 0 0, axis 0 0 1, limit lower=0 upper=0.8 effort=200 velocity=0.3
- added joint wrist_rotate_joint: type revolute, parent arm_extend_forearm, child arm_wrist_rot, origin xyz=0.18 0 0 rpy=0 0 0, axis 1 0 0, limit lower=-1.57 upper=1.57 effort=40 velocity=1.5

Commit message: 获取相机数据

File: model/myrobotv52.urdf (robot description, URDF)
Before this commit: robot vehicle_blue, 18 links, 17 joints
Links:
- added link camera_link; visual box size=0.06 0.09 0.05
- added link camera_optical_frame
Joints:
- added joint camera_fixed_joint: type fixed, parent gripper_base, child camera_link, origin xyz=0.13 0 0 rpy=0 0 0
- added joint camera_optical_joint: type fixed, parent camera_link, child camera_optical_frame, origin xyz=0 0 0 rpy=-1.57079632679 0 -1.57079632679

Commit message: xiangji tiaozheng

File: model/myrobotv52.urdf (robot description, URDF)
Before this commit: robot vehicle_blue, 20 links, 19 joints
Joints:
- joint camera_fixed_joint: origin xyz=0.13 0 0 rpy=0 0 0 -> xyz=0.15 0 0.03 rpy=0 -0.2 0
